File: HW/Ethernet.kicad_sch (KiCad schematic)
At the start: 28 parts, among them J8 HR911105A, U2 RTL8201F, Y1 Crystal_GND24_Small

Commit message: Small fixes to HW
Parts:
- removed R23, R24, R25, R26: 49.9R, Resistor_SMD:R_0603_1608Metric, symbol Device:R
- added C17: 22n, Capacitor_SMD:C_0603_1608Metric, symbol Device:C
Connections:
- net +3V3: no longer C16.1, J8.4, J8.5
- net GND: now also C17.2
- new net: C16.1, J8.4
- new net: C17.1, J8.5
