File: HW/dock.kicad_pcb (KiCad board)
At the start: 4 copper layers, 95 x 82.5 mm, 77 parts, among them J1 te_m.2_b, J2 te_m.2_b, J3 USB_C_Recept_16Pin, J4 Raspberry_Pi_2_3, J5 Conn_01x06, J6 USB_A, J7 AudioJack3, J8 HR911105A, J9 HDMI_A, SW1 SW_Push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

Commit message: Small fixes to HW
Parts:
- added C17: 22n, Capacitor_SMD:C_0603_1608Metric, F.Cu at (153.2, 140.0)
- moved C15 14.3 mm to (205.8, 107.6), turned to 180 degrees
- moved U4 10.2 mm to (206.9, 111.4), turned to 90 degrees
- moved C16 1.81 mm to (153.2, 138.2)
- moved J7 1.06 mm to (199.3, 151.5), turned to 90 degrees
Connections:
- C16 pad 1: +3V3 -> Net-(C16-Pad1)
- J8 pad 4: +3V3 -> Net-(C16-Pad1)
- J8 pad 5: +3V3 -> Net-(C17-Pad1)
Routing:
- net +3V3: track 323.4 -> 340.6 mm
- net Net-(C16-Pad1): track 0.00 -> 13.4 mm
- net Net-(C17-Pad1): track 0.00 -> 11.6 mm
- net /Storage/SD_D2: track 32.5 -> 43.3 mm
- net /Storage/SD_D3: track 33.8 -> 43.5 mm
- net GNDA: track 95.6 -> 104.9 mm
- net Net-(C6-Pad1): track 26.8 -> 18.3 mm
- net /Storage/SD_CMD: track 37.3 -> 44.1 mm
- net /Storage/SD_DET: track 45.1 -> 40.8 mm
- net /Storage/SD_D1: track 38.6 -> 35.3 mm
- net /Storage/SD_CLK: track 40.7 -> 43.7 mm
- net /Storage/SD_D0: track 35.6 -> 34.1 mm
- net GND: track 117.1 -> 116.0 mm, vias 205 -> 214
- net Net-(C5-Pad1): track 15.2 -> 16.1 mm
